File: Schematics/Schematics.kicad_pcb (KiCad board)
At the start: 2 copper layers, 77.5 x 96.5 mm, 18 parts, among them J1 BAT, U1 TP4056, U2 BH1750, U3 BME688, U4 BU30TD3WG, U5 NRF52840-DONGLE, U6 LIS3DH

Commit message: Uploading Modified Schematic with PCB version 1
Parts:
- removed J1: BAT, custom:KLS5-18650-005
- added BT1: 3.7V Li-ion, custom:KLS5-18650-005, F.Cu at (147.3, 98.8)
- moved R1 7.68 mm to (100.3, 110.0), turned to 180 degrees
- moved C2 6.54 mm to (92.8, 85.1), turned to 0 degrees
- moved U4 3.41 mm to (93.5, 80.8)
- moved U6 3.05 mm to (135.6, 86.4)
- moved D1 2.50 mm to (88.1, 75.4)
- moved C1 1.61 mm to (94.5, 76.7)
- moved R3 1.02 mm to (113.0, 80.3)
- moved R4 1.02 mm to (113.0, 85.1)
- moved R2 0.92 mm to (92.7, 113.8)
- moved U1 0.51 mm to (133.3, 49.9)
Routing:
- net +3V0: track 0.00 -> 131.5 mm, vias 0 -> 4
- net /SDA: track 0.00 -> 100.1 mm
- net /SCL: track 0.00 -> 93.6 mm
- net Net-(D1-Pad1): track 0.00 -> 61.3 mm
- net /VBAT: track 0.00 -> 57.9 mm
- net VCC: track 0.00 -> 52.0 mm
- net /INT1: track 0.00 -> 34.6 mm, vias 0 -> 2
- net GND: track 0.00 -> 14.8 mm
- net Net-(R3-Pad2): track 0.00 -> 9.92 mm
- net VBUS: track 0.00 -> 5.43 mm
- added copper zone on B.Cu, net GND
