File: Schematics/Schematics_v9.kicad_pcb (KiCad board)
At the start: 2 copper layers, 85 x 90 mm, 18 parts, among them U1 TP4056, U2 BH1750, U3 BME688, U4 BU30TD3WG, U5 NRF52840-DONGLE, U6 LIS3DH

Commit message: Created new versions of the pcb and generated gerber/drill files
Parts:
- BT1: footprint custom:BHC-18650-1P -> custom:KLS5-18650-005
- moved BT1 0.15 mm to (166.9, 104.9)
Routing:
- net Net-(U1-Pad4): track 35.3 -> 34.6 mm
- net Net-(U1-Pad5): track 67.0 -> 67.6 mm
Other:
- board text added: "+"
- board text added: "-"
- board text added: "v1.0"
- board text removed: "Lyubomir Nachev"
- board text removed: "PCB v1.0"
