File: Schematics/Schematics_copy1.kicad_sch (KiCad schematic)
At the start: 19 parts, among them U1 TP4056, U2 BH1750, U3 BME688, U4 BU30TD3WG, U5 NRF52840-DONGLE, U6 LIS3DH

Commit message: Edited the pcb board of the vodesht_vyzel and did some small changes on the pcb of the main module
Parts:
- removed H5: MountingHole, custom:Slot, symbol Mechanical:MountingHole
- added BT?: 3.7V Li-ion, custom:BHC-18650-1P, symbol Device:Battery
- added C?: 1u, Capacitor_THT:C_Disc_D5.1mm_W3.2mm_P5.00mm, symbol Device:C
- added D?: 1N5817, Diode_THT:D_DO-41_SOD81_P10.16mm_Horizontal, symbol Diode:1N5817
- added U?: BME688, custom:BME688, symbol BME688:BME688
- added U?: TP4056, custom:TP4056-18650, symbol TP4056_module:TP4056
- added U?: LIS3DH, custom:LIS3DH, symbol LIS3DH:LIS3DH
- added U?: BH1750, custom:BH1750, symbol BH1750:BH1750
- added U?: BU30TD3WG, Package_TO_SOT_SMD:SOT-23-5, symbol BU30TD3WG:BU30TD3WG
