File: Schematics/vodesht_vyzel/vodesht_vyzel.kicad_pcb (KiCad board)
At the start: 2 copper layers, 81 x 59 mm, 7 parts, among them U1 SSD1306, U2 NODEMCU32S, U3 NRF52840-DONGLE

Commit message: Generated new gerber files for the leader_node pcb
Parts:
- moved H3 1.41 mm to (191.0, 71.0)
- moved G*** 1.00 mm to (132.5, 74.5)
- moved H1 1.00 mm to (119.0, 71.0)
Connections:
- U2 pad 5: Net-(U1-Pad3) -> unconnected-(U2-Pad5)
- U2 pad 6: Net-(U1-Pad4) -> unconnected-(U2-Pad6)
- U2 pad 7: unconnected-(U2-Pad7) -> Net-(U1-Pad3)
- U2 pad 8: unconnected-(U2-Pad8) -> Net-(U1-Pad4)
Routing:
- net Net-(U1-Pad4): track 15.6 -> 10.3 mm
- net Net-(U1-Pad3): track 15.3 -> 10.0 mm
Other:
- board size 81 x 59 mm -> 80 x 60 mm
Changed lines of the file:
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@@
   (net 6 "Net-(U1-Pad3)")
   (net 7 "unconnected-(U2-Pad4)")
-  (net 8 "unconnected-(U2-Pad7)")
-  (net 9 "unconnected-(U2-Pad8)")
+  (net 8 "unconnected-(U2-Pad5)")
+  (net 9 "unconnected-(U2-Pad6)")
   (net 10 "unconnected-(U2-Pad9)")
   (net 11 "unconnected-(U2-Pad10)")
@@
       (net 7 "unconnected-(U2-Pad4)") (pinfunction "SVN") (pintype "bidirectional+no_connect"))
     (pad "5" thru_hole circle (at -11.43 -15.08) (size 2 2) (drill 1) (layers *.Cu *.Mask)
-      (net 6 "Net-(U1-Pad3)") (pinfunction "P34") (pintype "bidirectional"))
+      (net 8 "unconnected-(U2-Pad5)") (pinfunction "P34") (pintype "bidirectional+no_connect"))
     (pad "6" thru_hole circle (at -11.43 -12.54) (size 2 2) (drill 1) (layers *.Cu *.Mask)
-      (net 5 "Net-(U1-Pad4)") (pinfunction "P35") (pintype "bidirectional"))
+      (net 9 "unconnected-(U2-Pad6)") (pinfunction "P35") (pintype "bidirectional+no_connect"))
     (pad "7" thru_hole circle (at -11.43 -10) (size 2 2) (drill 1) (layers *.Cu *.Mask)
-      (net 8 "unconnected-(U2-Pad7)") (pinfunction "P32") (pintype "bidirectional+no_connect"))
+      (net 6 "Net-(U1-Pad3)") (pinfunction "P32") (pintype "bidirectional"))
     (pad "8" thru_hole circle (at -11.43 -7.46) (size 2 2) (drill 1) (layers *.Cu *.Mask)
-      (net 9 "unconnected-(U2-Pad8)") (pinfunction "P33") (pintype "bidirectional+no_connect"))
+      (net 5 "Net-(U1-Pad4)") (pinfunction "P33") (pintype "bidirectional"))
     (pad "9" thru_hole circle (at -11.43 -4.92) (size 2 2) (drill 1) (layers *.Cu *.Mask)
       (net 10 "unconnected-(U2-Pad9)") (pinfunction "P25") (pintype "bidirectional+no_connect"))
@@
   )
   (footprint "MountingHole:MountingHole_2.5mm" (layer "F.Cu")
-    (at 119 72)
+    (at 119 71)
     (descr "Mounting Hole 2.5mm, no annular")
     (tags "mounting hole 2.5mm no annular")
@@
   )
   (footprint "LOGO" (layer "F.Cu")
-    (at 132.5 75.5)
+    (at 132.5 74.5)
     (attr board_only exclude_from_pos_files exclude_from_bom)
     (fp_text reference "G***" (at -9.5 -6) (layer "F.SilkS") hide
@@
   )
   (footprint "MountingHole:MountingHole_2.5mm" (layer "F.Cu")
-    (at 192 72 180)
+    (at 191 71 180)
     (descr "Mounting Hole 2.5mm, no annular")
     (tags "mounting hole 2.5mm no annular")
@@
     (pad "" np_thru_hole circle (at 0 0 180) (size 2.5 2.5) (drill 2.5) (layers *.Cu *.Mask))
   )
-  (gr_line (start 115 72) (end 115 123) (layer "Edge.Cuts") (width 0.1))
+  (gr_line (start 115 70) (end 115 124) (layer "Edge.Cuts") (width 0.1))
   (gr_line (start 174.5 124) (end 174.5 118.5) (layer "Edge.Cuts") (width 0.1))
   (gr_arc (start 174.5 124) (mid 173.62132 126.12132) (end 171.5 127) (layer "Edge.Cuts") (width 0.1))
-  (gr_line (start 119 127) (end 171.5 127) (layer "Edge.Cuts") (width 0.1))
-  (gr_line (start 193 115.5) (end 177.5 115.5) (layer "Edge.Cuts") (width 0.1))
-  (gr_arc (start 119 127) (mid 116.171573 125.828427) (end 115 123) (layer "Edge.Cuts") (width 0.1))
-  (gr_arc (start 115 72) (mid 116.171573 69.171573) (end 119 68) (layer "Edge.Cuts") (width 0.1))
+  (gr_line (start 118 127) (end 171.5 127) (layer "Edge.Cuts") (width 0.1))
+  (gr_arc (start 115 70) (mid 115.87868 67.87868) (end 118 67) (layer "Edge.Cuts") (width 0.1))
+  (gr_line (start 192 115.5) (end 177.5 115.5) (layer "Edge.Cuts") (width 0.1))
+  (gr_arc (start 195 112.5) (mid 194.12132 114.62132) (end 192 115.5) (layer "Edge.Cuts") (width 0.1))
+  (gr_arc (start 192 67) (mid 194.12132 67.87868) (end 195 70) (layer "Edge.Cuts") (width 0.1))
   (gr_arc (start 174.5 118.5) (mid 175.37868 116.37868) (end 177.5 115.5) (layer "Edge.Cuts") (width 0.1))
-  (gr_line (start 196 112.5) (end 196 72) (layer "Edge.Cuts") (width 0.1))
-  (gr_line (start 192 68) (end 119 68) (layer "Edge.Cuts") (width 0.1))
-  (gr_arc (start 196 112.5) (mid 195.12132 114.62132) (end 193 115.5) (layer "F.Fab") (width 0.1))
-  (gr_arc (start 192 68) (mid 194.828427 69.171573) (end 196 72) (layer "F.Fab") (width 0.1))
-  (gr_text "Lyubomir Nachev" (at 178 71) (layer "F.Cu")
+  (gr_line (start 195 112.5) (end 195 70) (layer "Edge.Cuts") (width 0.1))
+  (gr_arc (start 118 127) (mid 115.87868 126.12132) (end 115 124) (layer "Edge.Cuts") (width 0.1))
+  (gr_line (start 192 67) (end 118 67) (layer "Edge.Cuts") (width 0.1))
+  (gr_text "Lyubomir Nachev" (at 178 69.5) (layer "F.Cu")
     (effects (font (size 1.5 1.5) (thickness 0.3) italic))
   )
-  (gr_text "PCB v1.0" (at 183.5 74) (layer "F.Cu")
+  (gr_text "PCB v1.0" (at 182.5 72.5) (layer "F.Cu")
     (effects (font (size 1.5 1.5) (thickness 0.3) italic))
   )
   (dimension (type aligned) (layer "F.Fab")
-    (pts (xy 170 68) (xy 170 127))
-    (height -30.5)
-    (gr_text "59.0000 mm" (at 199.35 97.5 90) (layer "F.Fab")
+    (pts (xy 171.5 127) (xy 171.5 67))
+    (height 28.5)
+    (gr_text "60.0000 mm" (at 198.85 97 90) (layer "F.Fab")
       (effects (font (size 1 1) (thickness 0.15)))
     )
@@
   )
   (dimension (type aligned) (layer "F.Fab")
-    (pts (xy 115 72) (xy 196 72))
-    (height -9)
-    (gr_text "81.0000 mm" (at 155.5 61.85) (layer "F.Fab")
+    (pts (xy 115 70) (xy 195 70))
+    (height -8)
+    (gr_text "80.0000 mm" (at 155 60.85) (layer "F.Fab")
       (effects (font (size 1 1) (thickness 0.15)))
     )
@@
   (segment (start 143 81) (end 143 96.5) (width 0.5) (layer "F.Cu") (net 2))
   (segment (start 147.07 79.26) (end 147.07 76.93) (width 0.5) (layer "F.Cu") (net 2))
-  (segment (start 145 101.5) (end 144.19 102.31) (width 0.5) (layer "F.Cu") (net 5))
-  (segment (start 144.19 102.31) (end 141 102.31) (width 0.5) (layer "F.Cu") (net 5))
-  (segment (start 147.07 91.96) (end 145.54 91.96) (width 0.5) (layer "F.Cu") (net 5))
-  (segment (start 145 92.5) (end 145 101.5) (width 0.5) (layer "F.Cu") (net 5))
-  (segment (start 145.54 91.96) (end 145 92.5) (width 0.5) (layer "F.Cu") (net 5))
-  (segment (start 147.07 89.42) (end 145.08 89.42) (width 0.5) (layer "F.Cu") (net 6))
-  (segment (start 144 90.5) (end 144 99) (width 0.5) (layer "F.Cu") (net 6))
-  (segment (start 144 99) (end 143.23 99.77) (width 0.5) (layer "F.Cu") (net 6))
+  (segment (start 145 98) (end 145.96 97.04) (width 0.5) (layer "F.Cu") (net 5))
+  (segment (start 144.19 102.31) (end 145 101.5) (width 0.5) (layer "F.Cu") (net 5))
+  (segment (start 141 102.31) (end 144.19 102.31) (width 0.5) (layer "F.Cu") (net 5))
+  (segment (start 145 101.5) (end 145 98) (width 0.5) (layer "F.Cu") (net 5))
+  (segment (start 145.96 97.04) (end 147.07 97.04) (width 0.5) (layer "F.Cu") (net 5))
+  (segment (start 143.23 99.77) (end 144 99) (width 0.5) (layer "F.Cu") (net 6))
   (segment (start 141 99.77) (end 143.23 99.77) (width 0.5) (layer "F.Cu") (net 6))
-  (segment (start 145.08 89.42) (end 144 90.5) (width 0.5) (layer "F.Cu") (net 6))
+  (segment (start 144 96) (end 145.5 94.5) (width 0.5) (layer "F.Cu") (net 6))
+  (segment (start 144 99) (end 144 96) (width 0.5) (layer "F.Cu") (net 6))
+  (segment (start 145.5 94.5) (end 147.07 94.5) (width 0.5) (layer "F.Cu") (net 6))
   (segment (start 169.93 102.16) (end 171.84 102.16) (width 0.5) (layer "F.Cu") (net 27))
   (segment (start 172.5 99) (end 173.105 98.395) (width 0.5) (layer "F.Cu") (net 27))
